File: PCB/BSS138-level-shifter.kicad_sch (KiCad schematic)
At the start: 3 parts, among them Q1 BSS138

Commit message: Balthazar Thinkpad USB adapter v1.0
Parts:
- renumbered Q1 to Q2, R4 to R20, R11 to R21
