File: PCB/Thinkpad-USB-keyboard-PCB.kicad_pcb (KiCad board)
At the start: 2 copper layers, 111 x 64 mm, 95 parts, among them J1 USB_C_Receptacle_USB2.0, J2 USB_A, J3 USB_A, J4 SWD, J6 Conn_02x20_Odd_Even_MountingP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, J7 USB_C_Receptacle_USB2.0, Q1 BSS138, Q2 BSS138, Q3 BSS138, SW1 SW_Push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

Commit message: Balthazar Thinkpad USB adapter v1.0
Parts:
- removed C1, C18, C2, C20, C33: 10uF, Capacitor_SMD:C_1206_3216Metric_Pad1.33x1.80mm_HandSolder
- removed C10, C12, C13, C6, C7, C8: 100nF, Capacitor_SMD:C_0402_1005Metric_Pad0.74x0.62mm_HandSolder
- removed C3, C4: 18pF, Capacitor_SMD:C_0402_1005Metric_Pad0.74x0.62mm_HandSolder
- removed H5, H6, H7, H8: MountingHole_Pad, MountingHole:MountingHole_3.2mm_M3_ISO7380_Pad
- removed J2, J3: USB_A, Connector_USB:USB_A_Molex_67643_Horizontal
- removed J7: USB_C_Receptacle_USB2.0, Connector_USB:USB_C_Receptacle_HRO_TYPE-C-31-M-12
- removed R19: 1M, Resistor_SMD:R_0805_2012Metric_Pad1.20x1.40mm_HandSolder
- removed R5: 12k, Resistor_SMD:R_0805_2012Metric_Pad1.20x1.40mm_HandSolder
- removed R6, R7, R8, R9: 56k, Resistor_SMD:R_0805_2012Metric_Pad1.20x1.40mm_HandSolder
- removed U1, U4, U5: SRV05-4, Package_TO_SOT_SMD:SOT-23-6
- removed U3: USB2514B_Bi, Package_DFN_QFN:QFN-36-1EP_6x6mm_P0.5mm_EP3.7x3.7mm
- removed Y1: 24MHz, Crystal:Crystal_SMD_3225-4Pin_3.2x2.5mm_HandSoldering
- F1: value ASMD1206-150 -> 1812L075PR
- moved H2 80.7 mm to (64.7, 0.30)
- moved H11 60.2 mm to (21.0, 0.00)
- moved H4 58.8 mm to (64.7, 57.7)
- moved H3 55.8 mm to (11.3, 57.7)
- moved C15 52.2 mm to (44.1, 14.3), turned to 0 degrees
- moved H12 51.8 mm to (10.8, 29.8)
- moved H1 51.3 mm to (11.3, 0.30)
- moved C17 43.1 mm to (19.7, 7.40), turned to 90 degrees
- moved C14 43.0 mm to (36.9, 14.9)
- moved C16 43.0 mm to (37.0, 17.8)
- moved D4 43.0 mm to (33.2, 16.2)
- moved F1 43.0 mm to (37.6, 11.7)
- moved J1 43.0 mm to (43.0, 1.06)
- moved U10 43.0 mm to (43.5, 10.4)
- moved R1 43.0 mm to (46.7, 7.38)
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Connections:
- R13 pad 1: D2- -> DUP-
- R3 pad 1: D2+ -> DUP+
Routing:
- net +5V: track 250.3 -> 105.0 mm, vias 13 -> 5
- net D3-: track 66.6 -> 0.00 mm
- net D3+: track 65.0 -> 0.00 mm
- net +3V3: track 274.8 -> 211.5 mm, vias 18 -> 13
- net D1+: track 58.4 -> 0.00 mm
- net D1-: track 58.4 -> 0.00 mm
- net GND: track 93.6 -> 41.7 mm, vias 163 -> 63
- net /~{USB_BOOT}: track 11.3 -> 53.8 mm
- net D2-: track 33.9 -> 0.00 mm
- net D2+: track 31.0 -> 0.00 mm, vias 2 -> 0
- net D4-: track 28.6 -> 0.00 mm
- net D4+: track 27.7 -> 0.00 mm
- net DUP-: track 23.1 -> 40.9 mm, vias 0 -> 2
- net TP4-CLK-5V: track 11.4 -> 29.0 mm, vias 0 -> 2
- net DUP+: track 23.0 -> 40.2 mm, vias 0 -> 2
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- added copper zone on In1.Cu, net GND
- added copper zone on In2.Cu, net GND
- removed copper zone on B.Cu, net +3V3
- removed copper zone on F.Cu, net +3V3
- removed copper zone on B.Cu, net +5V
- removed copper zone on F.Cu, net +5V
- removed copper zone on B.Cu, net GNDPWR
- removed copper zone on F.Cu, net GNDPWR
Other:
- board size 111 x 64 mm -> 60 x 64 mm
- copper layers 2 -> 4
- board text added: "Balthazar Open Source NLNET 9/7/2024"
- board text added: "Thinkpad T410/etc keyboard to USB adapter"
- board text removed: "BOOT"
- board text removed: "Thinkpad T410/etc keyboard to USB adapter Pylon 1/15/2024"
